File: led-light-sensor/led-sensor-2.sch (KiCad schematic (older format))
At the start: 8 parts, among them J1 CONN_01X03, U1 LMC6482

Commit message: Convert to KiCad 5
Parts:
- C1: symbol C -> led-sensor-2-rescue:C-RESCUE-led-sensor-2
- D1: symbol LED -> led-sensor-2-rescue:LED-RESCUE-led-sensor-2
- J1: symbol CONN_01X03 -> led-sensor-2-rescue:CONN_01X03-RESCUE-led-sensor-2
- R1, R2, R3: symbol R -> led-sensor-2-rescue:R-RESCUE-led-sensor-2
- RV1: symbol POT -> led-sensor-2-rescue:POT-RESCUE-led-sensor-2
- U1: symbol LMC6482 -> led-sensor-2-rescue:LMC6482-RESCUE-led-sensor-2
Connections:
- wire segments 20 -> 26
Changed lines of the file:
@@
-EESchema Schematic File Version 2
-LIBS:74xgxx
-LIBS:74xx
-LIBS:ac-dc
-LIBS:actel
-LIBS:adc-dac
-LIBS:allegro
-LIBS:Altera
-LIBS:analog_devices
-LIBS:analog_switches
-LIBS:atmel
-LIBS:audio
-LIBS:battery_management
-LIBS:bbd
-LIBS:bosch
-LIBS:brooktre
-LIBS:cmos4000
-LIBS:cmos_ieee
-LIBS:conn
-LIBS:contrib
-LIBS:cypress
-LIBS:dc-dc
-LIBS:device
-LIBS:digital-audio
-LIBS:diode
-LIBS:display
-LIBS:dsp
-LIBS:elec-unifil
-LIBS:ESD_Protection
-LIBS:ftdi
-LIBS:gennum
-LIBS:graphic
-LIBS:hc11
-LIBS:infineon
-LIBS:intel
-LIBS:interface
-LIBS:intersil
-LIBS:ir
-LIBS:Lattice
-LIBS:leds
-LIBS:LEM
-LIBS:linear
-LIBS:logo
-LIBS:maxim
-LIBS:mechanical
-LIBS:memory
-LIBS:microchip
-LIBS:microchip_dspic33dsc
-LIBS:microchip_pic10mcu
-LIBS:microchip_pic12mcu
-LIBS:microchip_pic16mcu
-LIBS:microchip_pic18mcu
-LIBS:microchip_pic24mcu
-LIBS:microchip_pic32mcu
-LIBS:microcontrollers
-LIBS:modules
-LIBS:motor_drivers
-LIBS:motorola
-LIBS:motors
-LIBS:msp430
-LIBS:nordicsemi
-LIBS:nxp
-LIBS:nxp_armmcu
-LIBS:onsemi
-LIBS:opto
-LIBS:Oscillators
-LIBS:philips
-LIBS:power
-LIBS:Power_Management
-LIBS:powerint
-LIBS:pspice
-LIBS:references
-LIBS:regul
-LIBS:relays
-LIBS:rfcom
-LIBS:RFSolutions
-LIBS:sensors
-LIBS:silabs
-LIBS:siliconi
-LIBS:stm8
-LIBS:stm32
-LIBS:supertex
-LIBS:switches
-LIBS:texas
-LIBS:transf
-LIBS:transistors
-LIBS:triac_thyristor
-LIBS:ttl_ieee
-LIBS:valves
-LIBS:video
-LIBS:wiznet
-LIBS:Worldsemi
-LIBS:Xicor
-LIBS:xilinx
-LIBS:zetex
-LIBS:Zilog
+EESchema Schematic File Version 4
 LIBS:led-sensor-2-cache
 EELAYER 26 0
@@
 $EndDescr
 $Comp
-L LMC6482 U1
+L led-sensor-2-rescue:LMC6482-RESCUE-led-sensor-2 U1
 U 1 1 58FBD66A
 P 5350 3950
@@
 $EndComp
 $Comp
-L LMC6482 U1
+L led-sensor-2-rescue:LMC6482-RESCUE-led-sensor-2 U1
 U 2 1 58FBD66B
 P 6900 4050
@@
 $EndComp
 $Comp
-L R R1
+L led-sensor-2-rescue:R-RESCUE-led-sensor-2 R1
 U 1 1 58FBD66C
 P 4700 3850
@@
 $EndComp
 $Comp
-L R R3
+L led-sensor-2-rescue:R-RESCUE-led-sensor-2 R3
 U 1 1 58FBD66D
 P 5350 3200
@@
 $EndComp
 $Comp
-L R R2
+L led-sensor-2-rescue:R-RESCUE-led-sensor-2 R2
 U 1 1 58FBD66E
 P 4700 4350
@@
 $EndComp
 $Comp
-L LED D1
+L led-sensor-2-rescue:LED-RESCUE-led-sensor-2 D1
 U 1 1 58FBD66F
 P 4200 4350
@@
 $EndComp
 $Comp
-L GND #PWR01
+L led-sensor-2-rescue:GND-RESCUE-led-sensor-2 #PWR01
 U 1 1 58FBD670
 P 6800 4350
@@
 $EndComp
 $Comp
-L GND #PWR02
+L led-sensor-2-rescue:GND-RESCUE-led-sensor-2 #PWR02
 U 1 1 58FBD671
 P 4400 3850
@@
 $EndComp
 $Comp
-L C C1
+L led-sensor-2-rescue:C-RESCUE-led-sensor-2 C1
 U 1 1 58FBD672
 P 5350 2800
@@
 $EndComp
 $Comp
-L +3.3V #PWR03
+L led-sensor-2-rescue:+3.3V-RESCUE-led-sensor-2 #PWR03
 U 1 1 58FBD673
 P 6800 3750
@@
 $EndComp
 $Comp
-L GND #PWR04
+L led-sensor-2-rescue:GND-RESCUE-led-sensor-2 #PWR04
 U 1 1 58FBD674
 P 4450 4650
@@
 $EndComp
 $Comp
-L +3.3V #PWR05
+L led-sensor-2-rescue:+3.3V-RESCUE-led-sensor-2 #PWR05
 U 1 1 58FBD675
 P 5250 4250
@@
 $EndComp
 $Comp
-L GND #PWR06
+L led-sensor-2-rescue:GND-RESCUE-led-sensor-2 #PWR06
 U 1 1 58FBD676
 P 5250 3650
@@
 $EndComp
 $Comp
-L POT RV1
+L led-sensor-2-rescue:POT-RESCUE-led-sensor-2 RV1
 U 1 1 58FBD677
 P 6300 4150
@@
 $EndComp
 $Comp
-L GND #PWR07
+L led-sensor-2-rescue:GND-RESCUE-led-sensor-2 #PWR07
 U 1 1 58FBD678
 P 6300 4300
@@
 $EndComp
 $Comp
-L +3.3V #PWR08
+L led-sensor-2-rescue:+3.3V-RESCUE-led-sensor-2 #PWR08
 U 1 1 58FBD679
 P 6300 4000
@@
 $EndComp
 $Comp
-L CONN_01X03 J1
+L led-sensor-2-rescue:CONN_01X03-RESCUE-led-sensor-2 J1
 U 1 1 58FC2403
 P 4000 2900
@@
 $EndComp
 $Comp
-L GND #PWR09
+L led-sensor-2-rescue:GND-RESCUE-led-sensor-2 #PWR09
 U 1 1 58FC24F5
 P 4300 3000
@@
 $EndComp
 $Comp
-L +3.3V #PWR010
+L led-sensor-2-rescue:+3.3V-RESCUE-led-sensor-2 #PWR010
 U 1 1 58FC2512
 P 4300 2800
@@
 	4400 3850 4550 3850
 Wire Wire Line
-	4850 3850 5050 3850
+	4850 3850 4950 3850
 Wire Wire Line
 	4700 4200 4700 4050
 Wire Wire Line
-	4200 4050 5050 4050
+	4200 4050 4700 4050
 Wire Wire Line
 	4200 4050 4200 4200
@@
 	4200 4500 4200 4650
 Wire Wire Line
-	4200 4650 4700 4650
+	4200 4650 4450 4650
 Wire Wire Line
 	4700 4650 4700 4500
 Connection ~ 4450 4650
 Wire Wire Line
-	4950 2800 4950 3850
+	4950 2800 4950 3200
 Wire Wire Line
 	4950 2800 5200 2800
@@
 	5500 2800 5800 2800
 Wire Wire Line
-	5800 2800 5800 3950
+	5800 2800 5800 3200
 Wire Wire Line
 	5500 3200 5800 3200
@@
 Vout
 Wire Wire Line
-	5650 3950 6600 3950
+	5650 3950 5800 3950
 Wire Wire Line
 	6450 4150 6600 4150
+Wire Wire Line
+	4700 4050 5050 4050
+Wire Wire Line
+	4450 4650 4700 4650
+Wire Wire Line
+	4950 3850 5050 3850
+Wire Wire Line
+	4950 3200 4950 3850
+Wire Wire Line
+	5800 3200 5800 3950
+Wire Wire Line
+	5800 3950 6600 3950
 $EndSCHEMATC

Commit message: Update schematic
Parts:
- removed J1: CONN_01X03, Pin_Headers:Pin_Header_Straight_1x03_Pitch2.54mm, symbol led-sensor-2-rescue:CONN_01X03-RESCUE-led-sensor-2
- removed R1: 1k, Resistors_THT:R_Axial_DIN0309_L9.0mm_D3.2mm_P5.08mm_Vertical, symbol led-sensor-2-rescue:R-RESCUE-led-sensor-2
- removed R2: 1M, Resistors_THT:R_Axial_DIN0309_L9.0mm_D3.2mm_P5.08mm_Vertical, symbol led-sensor-2-rescue:R-RESCUE-led-sensor-2
- added C2: 1u, Capacitor_THT:C_Disc_D5.0mm_W2.5mm_P5.00mm, symbol Device:C
- added J1: Conn_01x03, Connector_PinHeader_2.54mm:PinHeader_1x03_P2.54mm_Vertical, symbol Connector_Generic:Conn_01x03
- added R1, R2: 10k, Resistor_THT:R_Axial_DIN0204_L3.6mm_D1.6mm_P5.08mm_Horizontal, symbol Device:R
- C1: value 1u -> 100n; footprint Capacitors_THT:C_Axial_L3.8mm_D2.6mm_P7.50mm_Horizontal -> Capacitor_THT:C_Disc_D5.0mm_W2.5mm_P5.00mm
- D1: footprint LEDs:LED_D5.0mm -> LED_THT:LED_D5.0mm
- R3: value 47k -> 5.1M; footprint Resistors_THT:R_Axial_DIN0309_L9.0mm_D3.2mm_P5.08mm_Vertical -> Resistor_THT:R_Axial_DIN0204_L3.6mm_D1.6mm_P5.08mm_Horizontal
- U1: footprint Housings_DIP:DIP-8_W7.62mm -> Package_DIP:DIP-8_W7.62mm
Connections:
- wire segments 26 -> 32
Other:
- moved on the sheet: C1, D1, R3, RV1, U1A, U1B

Commit message: Remove rescue symbols
Parts:
- C1: symbol led-sensor-2-rescue:C-RESCUE-led-sensor-2 -> Device:C
- D1: symbol led-sensor-2-rescue:LED-RESCUE-led-sensor-2 -> Device:LED
- R3: symbol led-sensor-2-rescue:R-RESCUE-led-sensor-2 -> Device:R
- RV1: symbol led-sensor-2-rescue:POT-RESCUE-led-sensor-2 -> Device:POT
- U1: symbol led-sensor-2-rescue:LMC6482-RESCUE-led-sensor-2 -> Amplifier_Operational:LMC6482
Connections:
- wire segments 32 -> 34
Changed lines of the file:
@@
 $EndDescr
 $Comp
-L led-sensor-2-rescue:LMC6482-RESCUE-led-sensor-2 U1
+L Amplifier_Operational:LMC6482 U1
 U 1 1 58FBD66A
 P 5300 3900
@@
 $EndComp
 $Comp
-L led-sensor-2-rescue:LMC6482-RESCUE-led-sensor-2 U1
+L Amplifier_Operational:LMC6482 U1
 U 2 1 58FBD66B
 P 7400 4000
@@
 $EndComp
 $Comp
-L led-sensor-2-rescue:R-RESCUE-led-sensor-2 R3
+L Device:R R3
 U 1 1 58FBD66D
 P 5300 5300
@@
 $EndComp
 $Comp
-L led-sensor-2-rescue:LED-RESCUE-led-sensor-2 D1
+L Device:LED D1
 U 1 1 58FBD66F
 P 3800 3350
@@
 $EndComp
 $Comp
-L led-sensor-2-rescue:GND-RESCUE-led-sensor-2 #PWR01
-U 1 1 58FBD670
-P 7300 4300
-F 0 "#PWR01" H 7300 4050 50  0001 C CNN
-F 1 "GND" H 7305 4127 50  0000 C CNN
-F 2 "" H 7300 4300 50  0001 C CNN
-F 3 "" H 7300 4300 50  0001 C CNN
-	1    7300 4300
-	1    0    0    -1
-$EndComp
-$Comp
-L led-sensor-2-rescue:C-RESCUE-led-sensor-2 C1
+L Device:C C1
 U 1 1 58FBD672
 P 5300 4900
@@
 $EndComp
 $Comp
-L led-sensor-2-rescue:+3.3V-RESCUE-led-sensor-2 #PWR03
+L power:+3.3V #PWR03
 U 1 1 58FBD673
 P 7300 3700
@@
 $EndComp
 $Comp
-L led-sensor-2-rescue:POT-RESCUE-led-sensor-2 RV1
+L Device:POT RV1
 U 1 1 58FBD677
 P 6500 4100
@@
 Vout
 $Comp
-L led-sensor-2-rescue:+3.3V-RESCUE-led-sensor-2 #PWR0101
+L power:+3.3V #PWR0101
 U 1 1 5ABA0602
 P 3800 2700
@@
 	5700 4900 5700 3900
 $Comp
-L led-sensor-2-rescue:GND-RESCUE-led-sensor-2 #PWR0102
-U 1 1 5ABA1F09
-P 5200 4200
-F 0 "#PWR0102" H 5200 3950 50  0001 C CNN
-F 1 "GND" H 5205 4027 50  0000 C CNN
-F 2 "" H 5200 4200 50  0001 C CNN
-F 3 "" H 5200 4200 50  0001 C CNN
-	1    5200 4200
-	1    0    0    -1
-$EndComp
-$Comp
-L led-sensor-2-rescue:+3.3V-RESCUE-led-sensor-2 #PWR0103
+L power:+3.3V #PWR0103
 U 1 1 5ABA1F22
 P 5200 3600
@@
 $EndComp
 $Comp
-L led-sensor-2-rescue:+3.3V-RESCUE-led-sensor-2 #PWR0104
+L power:+3.3V #PWR0104
 U 1 1 5ABA23CC
 P 4300 2700
@@
 	3800 4000 4900 4000
 Connection ~ 4900 4000
-$Comp
-L led-sensor-2-rescue:GND-RESCUE-led-sensor-2 #PWR0105
-U 1 1 5ABA3587
-P 4300 4800
-F 0 "#PWR0105" H 4300 4550 50  0001 C CNN
-F 1 "GND" H 4305 4627 50  0000 C CNN
-F 2 "" H 4300 4800 50  0001 C CNN
-F 3 "" H 4300 4800 50  0001 C CNN
-	1    4300 4800
-	1    0    0    -1
-$EndComp
 Wire Wire Line
 	4300 4800 4300 4500
 $Comp
-L led-sensor-2-rescue:GND-RESCUE-led-sensor-2 #PWR0106
-U 1 1 5ABA442C
-P 6500 4800
-F 0 "#PWR0106" H 6500 4550 50  0001 C CNN
-F 1 "GND" H 6505 4627 50  0000 C CNN
-F 2 "" H 6500 4800 50  0001 C CNN
-F 3 "" H 6500 4800 50  0001 C CNN
-	1    6500 4800
-	1    0    0    -1
-$EndComp
-$Comp
-L led-sensor-2-rescue:+3.3V-RESCUE-led-sensor-2 #PWR0107
+L power:+3.3V #PWR0107
 U 1 1 5ABA4449
 P 6500 3700
@@
 	2900 2900 2900 2850
 Wire Wire Line
-	2600 2900 2900 2900
+	2600 2900 2650 2900
 Wire Wire Line
 	2900 3100 2900 3150
 Wire Wire Line
-	2600 3100 2900 3100
+	2600 3100 2650 3100
 Wire Wire Line
 	3200 2850 2900 2850
@@
 Wire Wire Line
 	2900 3150 2900 3300
+$Comp
+L power:GND #PWR0102
+U 1 1 5ABA9325
+P 4300 4800
+F 0 "#PWR0102" H 4300 4550 50  0001 C CNN
+F 1 "GND" H 4305 4627 50  0000 C CNN
+F 2 "" H 4300 4800 50  0001 C CNN
+F 3 "" H 4300 4800 50  0001 C CNN
+	1    4300 4800
+	1    0    0    -1
+$EndComp
+$Comp
+L power:GND #PWR0105
+U 1 1 5ABA9344
+P 5200 4200
+F 0 "#PWR0105" H 5200 3950 50  0001 C CNN
+F 1 "GND" H 5205 4027 50  0000 C CNN
+F 2 "" H 5200 4200 50  0001 C CNN
+F 3 "" H 5200 4200 50  0001 C CNN
+	1    5200 4200
+	1    0    0    -1
+$EndComp
+$Comp
+L power:GND #PWR0106
+U 1 1 5ABA9363
+P 6500 4800
+F 0 "#PWR0106" H 6500 4550 50  0001 C CNN
+F 1 "GND" H 6505 4627 50  0000 C CNN
+F 2 "" H 6500 4800 50  0001 C CNN
+F 3 "" H 6500 4800 50  0001 C CNN
+	1    6500 4800
+	1    0    0    -1
+$EndComp
+$Comp
+L power:GND #PWR0108
+U 1 1 5ABA93F5
+P 7300 4300
+F 0 "#PWR0108" H 7300 4050 50  0001 C CNN
+F 1 "GND" H 7305 4127 50  0000 C CNN
+F 2 "" H 7300 4300 50  0001 C CNN
+F 3 "" H 7300 4300 50  0001 C CNN
+	1    7300 4300
+	1    0    0    -1
+$EndComp
+$Comp
+L power:PWR_FLAG #FLG0101
+U 1 1 5ABA91E7
+P 2650 2900
+F 0 "#FLG0101" H 2650 2975 50  0001 C CNN
+F 1 "PWR_FLAG" H 2650 3074 50  0000 C CNN
+F 2 "" H 2650 2900 50  0001 C CNN
+F 3 "" H 2650 2900 50  0001 C CNN
+	1    2650 2900
+	1    0    0    -1
+$EndComp
+Connection ~ 2650 2900
+Wire Wire Line
+	2650 2900 2900 2900
+$Comp
+L power:PWR_FLAG #FLG0102
+U 1 1 5ABA9242
+P 2650 3100
+F 0 "#FLG0102" H 2650 3175 50  0001 C CNN
+F 1 "PWR_FLAG" H 2650 3273 50  0000 C CNN
+F 2 "" H 2650 3100 50  0001 C CNN
+F 3 "" H 2650 3100 50  0001 C CNN
+	1    2650 3100
+	1    0    0    1
+$EndComp
+Connection ~ 2650 3100
+Wire Wire Line
+	2650 3100 2900 3100
 $EndSCHEMATC
