File: led-light-sensor/led-sensor-2.kicad_pcb (KiCad board)
At the start: 2 copper layers, 40.6 x 22.9 mm, 8 parts, among them J1 CONN_01X03, U1 LMC6482

Commit message: Update OtherMill design rules
Other:
- net class Default: clearance 0.82 -> 0.79375; trace_width 0.6 -> 0.79375; via_dia 0.83 -> 1.30175; via_drill 0.82 -> 0.79375
- rule trace_clearance: 0.82 -> 0.79375
- rule trace_min: 0.26 -> 0.254
- rule via_min_drill: 0.82 -> 0.79375
- rule via_min_size: 0.82 -> 1.30175
Changed lines of the file:
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@@
-(kicad_pcb (version 20170123) (host pcbnew "(2017-05-30 revision 8a82c9341)-master")
+(kicad_pcb (version 20190331) (host pcbnew "(5.1.0-73-g8985badc6)")
   (general
-    (links 17)
-    (no_connects 0)
-    (area 140.224999 46.3025 182.2025 73.038333)
     (thickness 1.54)
     (drawings 8)
@@
     (45 Margin user)
     (46 B.CrtYd user)
+    (47 F.CrtYd user)
     (48 B.Fab user)
   )
   (setup
-    (last_trace_width 0.6)
-    (trace_clearance 0.82)
+    (last_trace_width 0.79375)
+    (trace_clearance 0.79375)
     (zone_clearance 0.508)
     (zone_45_only no)
-    (trace_min 0.26)
+    (trace_min 0.254)
+    (via_size 1.30175)
+    (via_drill 0.79375)
+    (via_min_size 1.30175)
+    (via_min_drill 0.79375)
+    (uvia_size 0.3048)
+    (uvia_drill 0.254)
+    (uvias_allowed no)
+    (uvia_min_size 0.3048)
+    (uvia_min_drill 0.254)
+    (edge_width 0.15)
     (segment_width 0.2)
-    (edge_width 0.15)
-    (via_size 0.83)
-    (via_drill 0.82)
-    (via_min_size 0.82)
-    (via_min_drill 0.82)
-    (uvia_size 0.3)
-    (uvia_drill 0.1)
-    (uvias_allowed no)
-    (uvia_min_size 0.2)
-    (uvia_min_drill 0.1)
     (pcb_text_width 0.3)
     (pcb_text_size 1.5 1.5)
@@
       (layerselection 0x01000_7fffffff)
       (usegerberextensions false)
+      (usegerberattributes false)
+      (usegerberadvancedattributes false)
+      (creategerberjobfile false)
       (excludeedgelayer true)
       (linewidth 0.100000)
@@
       (hpglpennumber 1)
       (hpglpenspeed 20)
-      (hpglpendiameter 15)
+      (hpglpendiameter 15.000000)
       (psnegative false)
       (psa4output false)
@@
       (drillshape 0)
       (scaleselection 1)
-      (outputdirectory output/))
+      (outputdirectory "output/"))
   )
   (net 0 "")
@@
   (net 7 /Vout)
   (net_class Default "This is the default net class."
-    (clearance 0.82)
-    (trace_width 0.6)
-    (via_dia 0.83)
-    (via_drill 0.82)
-    (uvia_dia 0.3)
-    (uvia_drill 0.1)
-    (diff_pair_gap 0.82)
-    (diff_pair_width 0.26)
+    (clearance 0.79375)
+    (trace_width 0.79375)
+    (via_dia 1.30175)
+    (via_drill 0.79375)
+    (uvia_dia 0.3048)
+    (uvia_drill 0.254)
+    (diff_pair_width 0.254)
+    (diff_pair_gap 0.254)
     (add_net +3V3)
     (add_net /Vout)
@@
       (net 6 +3V3))
     (model Pin_Headers.3dshapes/Pin_Header_Straight_1x03_Pitch2.54mm.wrl
-      (at (xyz 0 -0.1 0))
+      (offset (xyz 0 -2.539999961853027 0))
       (scale (xyz 1 1 1))
       (rotate (xyz 0 0 90))
