File: phone_charger/phone_charger.sch (KiCad schematic (older format))
At the start: 19 parts, among them J1 Conn_01x02, J2 UE27AC54100, U1 ADP2302

Commit message: Phone charger assigned footprints
Parts:
- C1: footprint (none) -> Capacitors_SMD:C_1206_HandSoldering
- C2: footprint (none) -> Capacitors_SMD:C_0603_HandSoldering
- C3, C4: footprint (none) -> Capacitors_SMD:C_0805_HandSoldering
- D1: footprint (none) -> LEDs:LED_D3.0mm
- D2: footprint (none) -> Diodes_SMD:D_SOD-123
- D3: footprint (none) -> Diodes_SMD:D_SMB_Handsoldering
- F1: footprint (none) -> Fuse_Holders_and_Fuses:Fuse_SMD2920
- J1: footprint (none) -> Pin_Headers:Pin_Header_Straight_1x02_Pitch1.00mm
- J2: footprint digikey-footprints:USB_A_Female_UE27AC54100 -> phone_charger:USB_A_Female_SS-52100-001
- L1: footprint (none) -> phone_charger:L_TDK_VLF10040T-6R8N4R5
- R1: value R -> 300R; footprint (none) -> Resistors_THT:R_Axial_DIN0309_L9.0mm_D3.2mm_P12.70mm_Horizontal
- R2, R5, R7: footprint (none) -> Resistors_SMD:R_0603_HandSoldering
- R3, R4, R6: footprint (none) -> Resistors_SMD:R_0805_HandSoldering
- U1: footprint UJ_6 -> Housings_SOIC:SOIC-8-1EP_3.9x4.9mm_Pitch1.27mm
Changed lines of the file:
@@
 F 0 "L1" V 7440 1950 50  0000 C CNN
 F 1 "6.8u" V 7349 1950 50  0000 C CNN
-F 2 "" H 7250 1950 50  0001 C CNN
+F 2 "phone_charger:L_TDK_VLF10040T-6R8N4R5" H 7250 1950 50  0001 C CNN
 F 3 "" H 7250 1950 50  0001 C CNN
 	1    7250 1950
@@
 F 0 "C4" H 8000 2550 50  0000 L CNN
 F 1 "22u (16V)" H 8000 2450 50  0000 L CNN
-F 2 "" H 8038 2000 50  0001 C CNN
+F 2 "Capacitors_SMD:C_0805_HandSoldering" H 8038 2000 50  0001 C CNN
 F 3 "" H 8000 2150 50  0001 C CNN
 	1    8000 2150
@@
 F 0 "D3" V 6854 2179 50  0000 L CNN
 F 1 "B330B" V 6945 2179 50  0000 L CNN
-F 2 "" H 6900 2100 50  0001 C CNN
+F 2 "Diodes_SMD:D_SMB_Handsoldering" H 6900 2100 50  0001 C CNN
 F 3 "" H 6900 2100 50  0001 C CNN
 	1    6900 2100
@@
 F 0 "C2" H 6950 1950 50  0000 L CNN
 F 1 "0.1u (6.3V)" H 6950 1850 50  0000 L CNN
-F 2 "" H 6938 1600 50  0001 C CNN
+F 2 "Capacitors_SMD:C_0603_HandSoldering" H 6938 1600 50  0001 C CNN
 F 3 "" H 6900 1750 50  0001 C CNN
 	1    6900 1750
@@
 F 0 "C1" H 4815 1796 50  0000 L CNN
 F 1 "10u (25V)" H 4815 1705 50  0000 L CNN
-F 2 "" H 4738 1600 50  0001 C CNN
+F 2 "Capacitors_SMD:C_1206_HandSoldering" H 4738 1600 50  0001 C CNN
 F 3 "" H 4700 1750 50  0001 C CNN
 	1    4700 1750
@@
 F 0 "R2" H 5420 2146 50  0000 L CNN
 F 1 "100k" H 5420 2055 50  0000 L CNN
-F 2 "" V 5280 2100 50  0001 C CNN
+F 2 "Resistors_SMD:R_0603_HandSoldering" V 5280 2100 50  0001 C CNN
 F 3 "" H 5350 2100 50  0001 C CNN
 	1    5350 2100
@@
 F 0 "J2" H 6597 4690 60  0000 R CNN
 F 1 "UE27AC54100" H 6597 4796 60  0000 R CNN
-F 2 "digikey-footprints:USB_A_Female_UE27AC54100" H 6900 4950 60  0001 L CNN
+F 2 "phone_charger:USB_A_Female_SS-52100-001" H 6900 4950 60  0001 L CNN
 F 3 "https://www.amphenolcanada.com/ProductSearch/drawings/AC/UE27ACX4X0X.pdf" H 6900 5050 60  0001 L CNN
 F 4 "UE27AC54100-ND" H 6900 5150 60  0001 L CNN "Digi-Key_PN"
@@
 F 0 "R3" H 5570 4046 50  0000 L CNN
 F 1 "75k" H 5570 3955 50  0000 L CNN
-F 2 "" V 5430 4000 50  0001 C CNN
+F 2 "Resistors_SMD:R_0805_HandSoldering" V 5430 4000 50  0001 C CNN
 F 3 "~" H 5500 4000 50  0001 C CNN
 	1    5500 4000
@@
 F 0 "R4" H 5570 4546 50  0000 L CNN
 F 1 "50k" H 5570 4455 50  0000 L CNN
-F 2 "" V 5430 4500 50  0001 C CNN
+F 2 "Resistors_SMD:R_0805_HandSoldering" V 5430 4500 50  0001 C CNN
 F 3 "~" H 5500 4500 50  0001 C CNN
 	1    5500 4500
@@
 F 0 "R5" H 5570 5346 50  0000 L CNN
 F 1 "43k" H 5570 5255 50  0000 L CNN
-F 2 "" V 5430 5300 50  0001 C CNN
+F 2 "Resistors_SMD:R_0603_HandSoldering" V 5430 5300 50  0001 C CNN
 F 3 "~" H 5500 5300 50  0001 C CNN
 	1    5500 5300
@@
 F 0 "R6" H 5570 5846 50  0000 L CNN
 F 1 "50k" H 5570 5755 50  0000 L CNN
-F 2 "" V 5430 5800 50  0001 C CNN
+F 2 "Resistors_SMD:R_0805_HandSoldering" V 5430 5800 50  0001 C CNN
 F 3 "~" H 5500 5800 50  0001 C CNN
 	1    5500 5800
@@
 F 0 "R7" H 5850 5100 50  0000 L CNN
 F 1 "0R (OPT)" H 5850 5000 50  0000 L CNN
-F 2 "" V 5730 4800 50  0001 C CNN
+F 2 "Resistors_SMD:R_0603_HandSoldering" V 5730 4800 50  0001 C CNN
 F 3 "~" H 5800 4800 50  0001 C CNN
 	1    5800 4800
@@
 F 0 "F1" V 2625 1600 50  0000 C CNN
 F 1 "Polyfuse" V 2716 1600 50  0000 C CNN
-F 2 "" H 2900 1400 50  0001 L CNN
+F 2 "Fuse_Holders_and_Fuses:Fuse_SMD2920" H 2900 1400 50  0001 L CNN
 F 3 "~" H 2850 1600 50  0001 C CNN
 	1    2850 1600
@@
 F 0 "J1" H 2120 1817 50  0000 C CNN
 F 1 "Conn_01x02" H 2120 1726 50  0000 C CNN
-F 2 "" H 2200 1600 50  0001 C CNN
+F 2 "Pin_Headers:Pin_Header_Straight_1x02_Pitch1.00mm" H 2200 1600 50  0001 C CNN
 F 3 "~" H 2200 1600 50  0001 C CNN
 	1    2200 1600
@@
 F 0 "U1" H 6100 2687 60  0000 C CNN
 F 1 "ADP2302" H 6100 2581 60  0000 C CNN
-F 2 "UJ_6" H 6100 2600 60  0001 C CNN
+F 2 "Housings_SOIC:SOIC-8-1EP_3.9x4.9mm_Pitch1.27mm" H 6100 2600 60  0001 C CNN
 F 3 "" H 6100 1800 60  0000 C CNN
 	1    6100 1950
@@
 F 0 "C3" H 7550 2550 50  0000 L CNN
 F 1 "22u (16V)" H 7550 2450 50  0000 L CNN
-F 2 "" H 7588 2000 50  0001 C CNN
+F 2 "Capacitors_SMD:C_0805_HandSoldering" H 7588 2000 50  0001 C CNN
 F 3 "" H 7550 2150 50  0001 C CNN
 	1    7550 2150
@@
 F 0 "D2" H 3550 1384 50  0000 C CNN
 F 1 "D_Schottky" H 3550 1475 50  0000 C CNN
-F 2 "" H 3550 1600 50  0001 C CNN
+F 2 "Diodes_SMD:D_SOD-123" H 3550 1600 50  0001 C CNN
 F 3 "~" H 3550 1600 50  0001 C CNN
 	1    3550 1600
@@
 F 0 "D1" V 3038 4883 50  0000 R CNN
 F 1 "LED" V 2947 4883 50  0000 R CNN
-F 2 "" H 3000 5000 50  0001 C CNN
+F 2 "LEDs:LED_D3.0mm" H 3000 5000 50  0001 C CNN
 F 3 "~" H 3000 5000 50  0001 C CNN
 	1    3000 5000
@@
 P 3000 4550
 F 0 "R1" H 3070 4596 50  0000 L CNN
-F 1 "R" H 3070 4505 50  0000 L CNN
-F 2 "" V 2930 4550 50  0001 C CNN
+F 1 "300R" H 3070 4505 50  0000 L CNN
+F 2 "Resistors_THT:R_Axial_DIN0309_L9.0mm_D3.2mm_P12.70mm_Horizontal" V 2930 4550 50  0001 C CNN
 F 3 "~" H 3000 4550 50  0001 C CNN
 	1    3000 4550
