File: phone_charger/phone_charger.sch (KiCad schematic (older format))
At the start: 19 parts, among them J1 Conn_01x02, J2 SS-52100-001, U1 ADP2302

Commit message: Update fields
Parts:
- J2: Category Connectors, Interconnects -> (none); DK_Datasheet_Link https://www.amphenolcanada.com/ProductSearch/drawings/AC/UE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 -> (none); DK_Detail_Page /product-detail/en/amphenol-commercial-products/UE27AC54100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 -> (none); Description CONN RCPT USB TYPE A R/A GOLD -> (none); Digi-Key_PN UE27AC54100-ND -> 380-1412-ND; Family USB, DVI, HDMI Connectors -> (none); MPN UE27AC54100 -> SS-52100-001; Manufacturer Amphenol Commercial Products -> (none); Status Active -> (none)
Changed lines of the file:
@@
 F 1 "SS-52100-001" H 6497 4746 60  0000 R CNN
 F 2 "phone_charger:USB_A_Female_SS-52100-001" H 6800 4900 60  0001 L CNN
-F 3 "https://www.amphenolcanada.com/ProductSearch/drawings/AC/UE27ACX4X0X.pdf" H 6800 5000 60  0001 L CNN
-F 4 "UE27AC54100-ND" H 6800 5100 60  0001 L CNN "Digi-Key_PN"
-F 5 "UE27AC54100" H 6800 5200 60  0001 L CNN "MPN"
-F 6 "Connectors, Interconnects" H 6800 5300 60  0001 L CNN "Category"
-F 7 "USB, DVI, HDMI Connectors" H 6800 5400 60  0001 L CNN "Family"
-F 8 "https://www.amphenolcanada.com/ProductSearch/drawings/AC/UE27ACX4X0X.pdf" H 6800 5500 60  0001 L CNN "DK_Datasheet_Link"
-F 9 "/product-detail/en/amphenol-commercial-products/UE27AC54100/UE27AC54100-ND/1972253" H 6800 5600 60  0001 L CNN "DK_Detail_Page"
-F 10 "CONN RCPT USB TYPE A R/A GOLD" H 6800 5700 60  0001 L CNN "Description"
-F 11 "Amphenol Commercial Products" H 6800 5800 60  0001 L CNN "Manufacturer"
-F 12 "Active" H 6800 5900 60  0001 L CNN "Status"
+F 3 "https://belfuse.com/resources/drawings/stewartconnector/dr-stw-ss-52100-001.pdf" H 6800 5000 60  0001 L CNN
+F 4 "380-1412-ND" H 6600 4700 50  0001 C CNN "Digi-Key_PN"
+F 5 "SS-52100-001" H 6600 4700 50  0001 C CNN "MPN"
 	1    6600 4700
 	-1   0    0    1
