File: phone_charger/phone_charger.kicad_pcb (KiCad board)
At the start: 2 copper layers, 22.6 x 30.8 mm, 23 parts, among them J1 Conn_01x02, J2 SS-52100-001, U1 ADP2302

Commit message: Added some things to silkscreen
Other:
- board text added: "Top of USB"
Changed lines of the file:
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@@
-(kicad_pcb (version 20171130) (host pcbnew 5.0.2)
+(kicad_pcb (version 20171130) (host pcbnew "(5.0.0-3-g5ebb6b6)")
   (general
     (thickness 1.5748)
-    (drawings 8)
+    (drawings 12)
     (tracks 79)
     (zones 0)
@@
     (0 F.Cu signal)
     (31 B.Cu signal)
-    (32 B.Adhes user)
-    (33 F.Adhes user)
-    (34 B.Paste user)
-    (35 F.Paste user)
+    (32 B.Adhes user hide)
+    (33 F.Adhes user hide)
+    (34 B.Paste user hide)
+    (35 F.Paste user hide)
     (36 B.SilkS user)
     (37 F.SilkS user)
-    (38 B.Mask user)
-    (39 F.Mask user)
-    (40 Dwgs.User user)
-    (41 Cmts.User user)
-    (42 Eco1.User user)
-    (43 Eco2.User user)
+    (38 B.Mask user hide)
+    (39 F.Mask user hide)
+    (40 Dwgs.User user hide)
+    (41 Cmts.User user hide)
+    (42 Eco1.User user hide)
+    (43 Eco2.User user hide)
     (44 Edge.Cuts user)
-    (45 Margin user)
-    (46 B.CrtYd user)
-    (47 F.CrtYd user)
-    (48 B.Fab user)
-    (49 F.Fab user)
+    (45 Margin user hide)
+    (46 B.CrtYd user hide)
+    (47 F.CrtYd user hide)
+    (48 B.Fab user hide)
+    (49 F.Fab user hide)
   )
   (setup
@@
   (module phone_charger:USB_A_Female_SS-52100-001 (layer B.Cu)
     (at 101.092 56.134)
-    (fp_text reference J2 (at 0 0) (layer B.SilkS)
+    (fp_text reference J2 (at 0.127 0.762) (layer B.SilkS)
       (effects (font (size 1 1) (thickness 0.15)) (justify mirror))
     )
@@
     (descr "LED, diameter 3.0mm, 2 pins")
     (tags "LED diameter 3.0mm 2 pins")
-    (fp_text reference D1 (at -1.1176 -2.286) (layer B.SilkS)
+    (fp_text reference D1 (at -1.4986 -2.54) (layer B.SilkS)
       (effects (font (size 1 1) (thickness 0.15)) (justify mirror))
     )
@@
       (net 8 "Net-(F1-Pad2)"))
   )
+  (gr_text "Top of USB" (at 101.219 55.118) (layer B.SilkS)
+    (effects (font (size 1.5 1) (thickness 0.2)) (justify mirror))
+  )
+  (gr_line (start 88.646 58.039) (end 88.646 59.055) (layer B.SilkS) (width 0.2))
+  (gr_line (start 88.138 58.547) (end 89.154 58.547) (layer B.SilkS) (width 0.2))
+  (gr_line (start 90.932 58.293) (end 91.821 58.293) (layer B.SilkS) (width 0.2))
   (gr_text "Rev 2A" (at 108.458 72.39 90) (layer B.SilkS)
     (effects (font (size 1.016 1.016) (thickness 0.254)) (justify mirror))
