File: microcontroller/microcontroller.kicad_pcb (KiCad board)
At the start: 2 copper layers, 69.1 x 77.1 mm, 39 parts, among them J1 Conn_01x06_Male, J2 USB_B_Micro, Q1 MURATA-FILTER_CSTCR, SW1 SW_Push, SW2 SW_Push, U1 AP7312, U11 SD-105162, U6 F552X---PN80, U7 ICM-20689, X1 MS3V-T1R

Commit message: Updated assignment and overhauled part of solution
Parts:
- moved U11 56.3 mm to (112.8, 136.2), turned to 0 degrees
- moved J2 10.3 mm to (167.2, 110.9)
- moved C20 7.52 mm to (105.2, 114.4)
- moved C19 7.52 mm to (108.6, 111.3)
- moved C21 7.52 mm to (105.0, 108.5)
- moved C22 7.52 mm to (105.0, 111.5)
- moved SW1 7.52 mm to (112.1, 120.8)
- moved SW2 7.52 mm to (115.6, 113.2)
- moved U7 7.52 mm to (113.0, 108.8)
Routing:
- net +3V3: track 211.6 -> 158.2 mm
- net /MISO: track 130.4 -> 83.3 mm
- net /MOSI: track 127.2 -> 80.3 mm
- net /CS_SD: track 74.7 -> 28.9 mm
- net /SCK: track 125.1 -> 85.9 mm
- net +5V: track 77.5 -> 58.2 mm
- net /DET_SD: track 57.6 -> 43.4 mm
- net GND: track 64.9 -> 78.0 mm, vias 79 -> 57
- net Net-(R10-Pad1): track 57.8 -> 46.8 mm, vias 3 -> 1
- net /~RST: track 77.4 -> 70.2 mm
- net /D-: track 29.3 -> 22.9 mm
- net /D+: track 20.5 -> 14.2 mm
- net /CS_ICM: track 32.8 -> 36.7 mm
- net /INT_ICM: track 37.7 -> 40.6 mm
- net /TARGET_DP: track 22.8 -> 23.5 mm
Other:
- board size 69.1 x 77.1 mm -> 69.1 x 48.1 mm
