File: micro_assignment/micro_assignment.sch (KiCad schematic (older format))
At the start: 39 parts, among them J1 Conn_01x06_Male, J2 USB_B_Micro, Q1 MURATA-FILTER_CSTCR, SW1 SW_Push, SW2 SW_Push, U1 AP7312, U11 SD-105162, U6 F552X---PN80, U7 ICM-20689, X1 MS3V-T1R

Commit message: Updated assignment and overhauled part of solution
Parts:
- removed C19: 470n, Capacitor_SMD:C_0805_2012Metric_Pad1.15x1.40mm_HandSolder, symbol Device:C
- removed C20: 2u2, Capacitor_SMD:C_0805_2012Metric_Pad1.15x1.40mm_HandSolder, symbol Device:C
- removed C21: 100n, Capacitor_SMD:C_0805_2012Metric_Pad1.15x1.40mm_HandSolder, symbol Device:C
- removed C22: 10n, Capacitor_SMD:C_0805_2012Metric_Pad1.15x1.40mm_HandSolder, symbol Device:C
- removed U11: SD-105162, micro:SD-105162, symbol symbols:SD-105162
- removed U7: ICM-20689, Housings_DFN_QFN:QFN-24-1EP_4x4mm_Pitch0.5mm, symbol symbols:ICM-20689
- C1, C2, C3, C4, C5: footprint Capacitors_SMD:C_0402 -> (none)
- C10, C12, C13, C15, C16, C18, C6, C7, C8: footprint Capacitor_SMD:C_0805_2012Metric_Pad1.15x1.40mm_HandSolder -> (none)
- C17: footprint v02:C_SMD_WURTH_865080540002 -> (none)
- C9: footprint micro:153CLV-0405 -> (none)
- D1: footprint LEDs:LED_0805_HandSoldering -> (none)
- J1: footprint Pin_Headers:Pin_Header_Straight_1x06_Pitch2.54mm -> (none)
- J2: footprint Connectors_USB:USB_Micro-B_Molex-105017-0001 -> (none)
- Q1: footprint micro:MURATA-CSTCR_G -> (none)
- R1, R2: footprint Resistor_SMD:R_0402_1005Metric -> (none)
- R10, R11, R12, R4, R5, R9: footprint Resistor_SMD:R_0805_2012Metric_Pad1.15x1.40mm_HandSolder -> (none)
- SW1, SW2: footprint Buttons_Switches_THT:SW_PUSH_6mm -> (none)
- U1: footprint micro:SOT26 -> (none)
- U6: footprint Housings_QFP:LQFP-80_12x12mm_Pitch0.5mm -> (none)
- X1: footprint micro:MS3V-T1R -> (none)
Connections:
- wire segments 182 -> 141
Other:
- moved on the sheet: C1, C2, C3, C4, C5, J1, J2, R1, R2, U1

Commit message: renaming micro and making the footprints assigned for assignment version of the layout
Parts:
- C1, C10, C12, C13, C15, C16, C18, C4, C5, C6, C7, C8: footprint (none) -> Capacitor_SMD:C_0805_2012Metric_Pad1.15x1.40mm_HandSolder
- C17: footprint (none) -> micro:C_SMD_WURTH_865080540002
- C2, C3: footprint (none) -> Capacitor_SMD:C_0402_1005Metric
- C9: footprint (none) -> micro:153CLV-0405
- D1: footprint (none) -> LED_SMD:LED_0805_2012Metric_Pad1.15x1.40mm_HandSolder
- J1: footprint (none) -> Connector_PinHeader_2.54mm:PinHeader_1x06_P2.54mm_Vertical
- J2: footprint (none) -> Connector_USB:USB_Micro-B_Molex-105017-0001
- Q1: footprint (none) -> micro:MURATA-CSTCR_G; symbol symbols:MURATA-FILTER_CSTCR -> micro:MURATA-FILTER_CSTCR
- R1, R2: footprint (none) -> Resistor_SMD:R_0402_1005Metric
- R10, R11, R12, R4, R5, R9: footprint (none) -> Resistor_SMD:R_0805_2012Metric_Pad1.15x1.40mm_HandSolder
- SW1, SW2: footprint (none) -> Button_Switch_THT:SW_PUSH_6mm
- U1: footprint (none) -> micro:SOT26; symbol symbols:AP7312 -> micro:AP7312
- U6: footprint (none) -> Package_QFP:LQFP-80_12x12mm_P0.5mm; symbol symbols:F552X---PN80 -> micro:F552X---PN80
- X1: footprint (none) -> micro:MS3V-T1R; symbol symbols:MS3V-T1R -> micro:MS3V-T1R
Connections:
- wire segments 141 -> 139
Changed lines of the file:
@@
 	3900 3150 3600 3150
 $Comp
-L symbols:AP7312 U1
+L micro:AP7312 U1
 U 1 0 E58315B9
 P 2800 2950
 F 0 "U1" H 2400 3150 85  0000 L BNN
 F 1 "AP7312" H 2400 2650 85  0000 L BNN
-F 2 "" H 2800 2950 50  0001 C CNN
+F 2 "micro:SOT26" H 2800 2950 50  0001 C CNN
 F 3 "" H 2800 2950 50  0001 C CNN
 	1    2800 2950
@@
 $EndComp
 $Comp
-L symbols:MURATA-FILTER_CSTCR Q1
+L micro:MURATA-FILTER_CSTCR Q1
 U 1 1 5BF6A329
 P 8750 1500
 F 0 "Q1" H 8750 1786 59  0000 C CNN
 F 1 "MURATA-FILTER_CSTCR" H 8750 1681 59  0000 C CNN
-F 2 "" H 8750 1500 50  0001 C CNN
+F 2 "micro:MURATA-CSTCR_G" H 8750 1500 50  0001 C CNN
 F 3 "" H 8750 1500 50  0001 C CNN
 	1    8750 1500
@@
 $EndComp
 $Comp
-L symbols:MS3V-T1R X1
+L micro:MS3V-T1R X1
 U 1 1 5BF6CEEC
 P 6700 4500
 F 0 "X1" H 6750 4300 34  0000 C CNN
 F 1 "MS3V-T1R" H 6750 4250 34  0000 C CNN
-F 2 "" H 6700 4500 50  0001 C CNN
+F 2 "micro:MS3V-T1R" H 6700 4500 50  0001 C CNN
 F 3 "" H 6700 4500 50  0001 C CNN
 	1    6700 4500
@@
 F 0 "R4" H 5920 4146 50  0000 L CNN
 F 1 "0R" H 5920 4055 50  0000 L CNN
-F 2 "" V 5780 4100 50  0001 C CNN
+F 2 "Resistor_SMD:R_0805_2012Metric_Pad1.15x1.40mm_HandSolder" V 5780 4100 50  0001 C CNN
 F 3 "" H 5850 4100 50  0001 C CNN
 	1    5850 4100
@@
 F 0 "C7" V 6098 4400 50  0000 C CNN
 F 1 "12p" V 6189 4400 50  0000 C CNN
-F 2 "" H 6388 4250 50  0001 C CNN
+F 2 "Capacitor_SMD:C_0805_2012Metric_Pad1.15x1.40mm_HandSolder" H 6388 4250 50  0001 C CNN
 F 3 "" H 6350 4400 50  0001 C CNN
 	1    6350 4400
@@
 F 0 "C8" V 6500 4600 50  0000 C CNN
 F 1 "12p" V 6600 4600 50  0000 C CNN
-F 2 "" H 6388 4450 50  0001 C CNN
+F 2 "Capacitor_SMD:C_0805_2012Metric_Pad1.15x1.40mm_HandSolder" H 6388 4450 50  0001 C CNN
 F 3 "" H 6350 4600 50  0001 C CNN
 	1    6350 4600
@@
 F 0 "C13" H 7185 5504 50  0000 R CNN
 F 1 "470n" H 7185 5595 50  0000 R CNN
-F 2 "" H 7338 5400 50  0001 C CNN
+F 2 "Capacitor_SMD:C_0805_2012Metric_Pad1.15x1.40mm_HandSolder" H 7338 5400 50  0001 C CNN
 F 3 "" H 7300 5550 50  0001 C CNN
 	1    7300 5550
@@
 F 0 "C10" H 7065 5296 50  0000 L CNN
 F 1 "100n" H 7065 5205 50  0000 L CNN
-F 2 "" H 6988 5100 50  0001 C CNN
+F 2 "Capacitor_SMD:C_0805_2012Metric_Pad1.15x1.40mm_HandSolder" H 6988 5100 50  0001 C CNN
 F 3 "" H 6950 5250 50  0001 C CNN
 	1    6950 5250
@@
 F 0 "R10" H 11020 2046 50  0000 L CNN
 F 1 "100R" H 11020 1955 50  0000 L CNN
-F 2 "" V 10880 2000 50  0001 C CNN
+F 2 "Resistor_SMD:R_0805_2012Metric_Pad1.15x1.40mm_HandSolder" V 10880 2000 50  0001 C CNN
 F 3 "" H 10950 2000 50  0001 C CNN
 	1    10950 2000
@@
 F 0 "C12" H 7165 2646 50  0000 L CNN
 F 1 "1n" H 7165 2555 50  0000 L CNN
-F 2 "" H 7088 2450 50  0001 C CNN
+F 2 "Capacitor_SMD:C_0805_2012Metric_Pad1.15x1.40mm_HandSolder" H 7088 2450 50  0001 C CNN
 F 3 "" H 7050 2600 50  0001 C CNN
 	1    7050 2600
@@
 F 0 "C15" H 9250 1800 50  0000 L CNN
 F 1 "220n" H 9250 1700 50  0000 L CNN
-F 2 "" H 9388 1850 50  0001 C CNN
+F 2 "Capacitor_SMD:C_0805_2012Metric_Pad1.15x1.40mm_HandSolder" H 9388 1850 50  0001 C CNN
 F 3 "" H 9350 2000 50  0001 C CNN
 	1    9350 2000
@@
 F 0 "C16" H 9565 1746 50  0000 L CNN
 F 1 "220n" H 9565 1655 50  0000 L CNN
-F 2 "" H 9488 1550 50  0001 C CNN
+F 2 "Capacitor_SMD:C_0805_2012Metric_Pad1.15x1.40mm_HandSolder" H 9488 1550 50  0001 C CNN
 F 3 "" H 9450 1700 50  0001 C CNN
 	1    9450 1700
@@
 F 0 "C9" H 6450 5300 50  0000 L CNN
 F 1 "10u" H 6400 5200 50  0000 L CNN
-F 2 "" H 6688 5100 50  0001 C CNN
+F 2 "micro:153CLV-0405" H 6688 5100 50  0001 C CNN
 F 3 "" H 6650 5250 50  0001 C CNN
 	1    6650 5250
@@
 F 0 "C17" V 9900 1900 50  0000 C CNN
 F 1 "4u7" V 9800 1900 50  0000 C CNN
-F 2 "" H 9788 1900 50  0001 C CNN
+F 2 "micro:C_SMD_WURTH_865080540002" H 9788 1900 50  0001 C CNN
 F 3 "" H 9750 2050 50  0001 C CNN
 	1    9750 2050
@@
 F 0 "R5" H 7120 2146 50  0000 L CNN
 F 1 "47k" H 7120 2055 50  0000 L CNN
-F 2 "" V 6980 2100 50  0001 C CNN
+F 2 "Resistor_SMD:R_0805_2012Metric_Pad1.15x1.40mm_HandSolder" V 6980 2100 50  0001 C CNN
 F 3 "" H 7050 2100 50  0001 C CNN
 	1    7050 2100
@@
 F 0 "R11" H 11020 2546 50  0000 L CNN
 F 1 "1M" H 11020 2455 50  0000 L CNN
-F 2 "" V 10880 2500 50  0001 C CNN
+F 2 "Resistor_SMD:R_0805_2012Metric_Pad1.15x1.40mm_HandSolder" V 10880 2500 50  0001 C CNN
 F 3 "" H 10950 2500 50  0001 C CNN
 	1    10950 2500
@@
 F 0 "C18" H 11365 4596 50  0000 L CNN
 F 1 "100n" H 11365 4505 50  0000 L CNN
-F 2 "" H 11288 4400 50  0001 C CNN
+F 2 "Capacitor_SMD:C_0805_2012Metric_Pad1.15x1.40mm_HandSolder" H 11288 4400 50  0001 C CNN
 F 3 "" H 11250 4550 50  0001 C CNN
 	1    11250 4550
@@
 F 0 "R1" H 2020 4346 50  0000 L CNN
 F 1 "27R" H 2020 4255 50  0000 L CNN
-F 2 "" V 1880 4300 50  0001 C CNN
+F 2 "Resistor_SMD:R_0402_1005Metric" V 1880 4300 50  0001 C CNN
 F 3 "" H 1950 4300 50  0001 C CNN
 	1    1950 4300
@@
 F 0 "R2" H 2470 4446 50  0000 L CNN
 F 1 "27R" H 2470 4355 50  0000 L CNN
-F 2 "" V 2330 4400 50  0001 C CNN
+F 2 "Resistor_SMD:R_0402_1005Metric" V 2330 4400 50  0001 C CNN
 F 3 "" H 2400 4400 50  0001 C CNN
 	1    2400 4400
@@
 F 0 "C2" H 1865 4846 50  0000 L CNN
 F 1 "10p" H 1865 4755 50  0000 L CNN
-F 2 "" H 1788 4650 50  0001 C CNN
+F 2 "Capacitor_SMD:C_0402_1005Metric" H 1788 4650 50  0001 C CNN
 F 3 "" H 1750 4800 50  0001 C CNN
 	1    1750 4800
@@
 F 0 "C3" H 2265 4846 50  0000 L CNN
 F 1 "10p" H 2265 4755 50  0000 L CNN
-F 2 "" H 2188 4650 50  0001 C CNN
+F 2 "Capacitor_SMD:C_0402_1005Metric" H 2188 4650 50  0001 C CNN
 F 3 "" H 2150 4800 50  0001 C CNN
 	1    2150 4800
@@
 F 0 "R9" H 10370 2346 50  0000 L CNN
 F 1 "1k4" H 10370 2255 50  0000 L CNN
-F 2 "" V 10230 2300 50  0001 C CNN
+F 2 "Resistor_SMD:R_0805_2012Metric_Pad1.15x1.40mm_HandSolder" V 10230 2300 50  0001 C CNN
 F 3 "" H 10300 2300 50  0001 C CNN
 	1    10300 2300
@@
 F 0 "R12" H 11320 5446 50  0000 L CNN
 F 1 "300R" H 11320 5355 50  0000 L CNN
-F 2 "" V 11180 5400 50  0001 C CNN
+F 2 "Resistor_SMD:R_0805_2012Metric_Pad1.15x1.40mm_HandSolder" V 11180 5400 50  0001 C CNN
 F 3 "" H 11250 5400 50  0001 C CNN
 	1    11250 5400
@@
 F 0 "D1" V 11288 5683 50  0000 R CNN
 F 1 "LED" V 11197 5683 50  0000 R CNN
-F 2 "" H 11250 5800 50  0001 C CNN
+F 2 "LED_SMD:LED_0805_2012Metric_Pad1.15x1.40mm_HandSolder" H 11250 5800 50  0001 C CNN
 F 3 "" H 11250 5800 50  0001 C CNN
 	1    11250 5800
@@
 F 0 "C6" H 5965 4546 50  0000 L CNN
 F 1 "100n" H 5965 4455 50  0000 L CNN
-F 2 "" H 5888 4350 50  0001 C CNN
+F 2 "Capacitor_SMD:C_0805_2012Metric_Pad1.15x1.40mm_HandSolder" H 5888 4350 50  0001 C CNN
 F 3 "" H 5850 4500 50  0001 C CNN
 	1    5850 4500
@@
 Text Label 10650 5000 0    50   ~ 0
 DET_SD
-Wire Wire Line
-	6500 4400 6700 4400
-Wire Wire Line
-	6500 4600 6700 4600
 Wire Wire Line
 	2100 4300 3400 4300
@@
 F 0 "C1" H 1765 3146 50  0000 L CNN
 F 1 "1u" H 1765 3055 50  0000 L CNN
-F 2 "" H 1688 2950 50  0001 C CNN
+F 2 "Capacitor_SMD:C_0805_2012Metric_Pad1.15x1.40mm_HandSolder" H 1688 2950 50  0001 C CNN
 F 3 "" H 1650 3100 50  0001 C CNN
 	1    1650 3100
@@
 F 0 "C4" H 3715 3346 50  0000 L CNN
 F 1 "100n" H 3715 3255 50  0000 L CNN
-F 2 "" H 3638 3150 50  0001 C CNN
+F 2 "Capacitor_SMD:C_0805_2012Metric_Pad1.15x1.40mm_HandSolder" H 3638 3150 50  0001 C CNN
 F 3 "" H 3600 3300 50  0001 C CNN
 	1    3600 3300
@@
 F 0 "C5" H 4015 3346 50  0000 L CNN
 F 1 "1u" H 4015 3255 50  0000 L CNN
-F 2 "" H 3938 3150 50  0001 C CNN
+F 2 "Capacitor_SMD:C_0805_2012Metric_Pad1.15x1.40mm_HandSolder" H 3938 3150 50  0001 C CNN
 F 3 "" H 3900 3300 50  0001 C CNN
 	1    3900 3300
@@
 Wire Wire Line
 	7050 2750 7500 2750
-Connection ~ 6700 4400
-Wire Wire Line
-	6700 4400 6850 4400
-Connection ~ 6700 4600
-Wire Wire Line
-	6700 4600 7350 4600
 $Comp
 L Switch:SW_Push SW2
@@
 F 0 "SW2" V 10904 1698 50  0000 L CNN
 F 1 "SW_Push" V 10995 1698 50  0000 L CNN
-F 2 "" H 10950 1750 50  0001 C CNN
+F 2 "Button_Switch_THT:SW_PUSH_6mm" H 10950 1750 50  0001 C CNN
 F 3 "" H 10950 1750 50  0001 C CNN
 	1    10950 1550
@@
 F 0 "SW1" V 7454 2698 50  0000 L CNN
 F 1 "SW_Push" V 7545 2698 50  0000 L CNN
-F 2 "" H 7500 2750 50  0001 C CNN
+F 2 "Button_Switch_THT:SW_PUSH_6mm" H 7500 2750 50  0001 C CNN
 F 3 "" H 7500 2750 50  0001 C CNN
 	1    7500 2550
@@
 Connection ~ 7500 2350
 $Comp
-L symbols:F552X---PN80 U6
+L micro:F552X---PN80 U6
 U 1 1 5BF68EDA
 P 8950 4200
 F 0 "U6" H 8900 4250 150 0000 L CNN
 F 1 "F552X---PN80" H 8950 4200 50  0001 C CNN
-F 2 "" H 8950 4200 50  0001 C CNN
+F 2 "Package_QFP:LQFP-80_12x12mm_P0.5mm" H 8950 4200 50  0001 C CNN
 F 3 "" H 8950 4200 50  0001 C CNN
 	1    8950 4200
@@
 F 0 "J1" H 1956 6328 50  0000 C CNN
 F 1 "Conn_01x06_Male" H 1956 6237 50  0000 C CNN
-F 2 "" H 1850 5950 50  0001 C CNN
+F 2 "Connector_PinHeader_2.54mm:PinHeader_1x06_P2.54mm_Vertical" H 1850 5950 50  0001 C CNN
 F 3 "" H 1850 5950 50  0001 C CNN
 	1    1850 5950
@@
 F 0 "J2" H 1855 2167 50  0000 C CNN
 F 1 "USB_B_Micro" H 1855 2076 50  0000 C CNN
-F 2 "" H 1950 1650 50  0001 C CNN
+F 2 "Connector_USB:USB_Micro-B_Molex-105017-0001" H 1950 1650 50  0001 C CNN
 F 3 "" H 1950 1650 50  0001 C CNN
 	1    1800 1700
@@
 Wire Wire Line
 	2400 1350 2400 1500
+Wire Wire Line
+	6500 4400 6850 4400
+Wire Wire Line
+	6500 4600 7350 4600
 $EndSCHEMATC

Commit message: Removed net labels from microcontroller assignment schematic
Connections:
- net labels removed: CS_ICM, CS_SD, DET_SD, INT_ICM, MISO, MOSI, SCK, SCL, SDA, STE
- wire segments 139 -> 129
Changed lines of the file:
@@
 VUSB
-Wire Wire Line
-	10650 5300 11050 5300
-Text Label 9550 6300 1    50   ~ 0
-SCK
-Text Label 9950 6300 1    50   ~ 0
-MOSI
-Text Label 10650 5300 0    50   ~ 0
-MISO
 Wire Wire Line
 	10650 4300 11050 4300
@@
 Text Label 10650 4200 0    50   ~ 0
 RXD
-Text Label 9650 6300 1    50   ~ 0
-SDA
-Text Label 9750 6300 1    50   ~ 0
-SCL
-Text Label 9850 6300 1    50   ~ 0
-STE
 Wire Wire Line
 	8350 2700 8350 2500
@@
 Wire Wire Line
 	8950 2700 8950 2500
-Text Label 6950 4900 0    50   ~ 0
-CS_SD
 Wire Wire Line
 	7350 4500 6850 4500
@@
 	6200 4700 7350 4700
 Wire Wire Line
-	7350 4900 6950 4900
-Wire Wire Line
 	7000 4300 7000 4400
 Wire Wire Line
 	7000 4400 7350 4400
-Wire Wire Line
-	7350 4200 7050 4200
-Wire Wire Line
-	7350 4100 7050 4100
-Wire Wire Line
-	10650 5000 11050 5000
-Text Label 7050 4200 0    50   ~ 0
-INT_ICM
-Wire Wire Line
-	9550 6000 9550 6300
-Wire Wire Line
-	9650 6000 9650 6300
-Wire Wire Line
-	9750 6000 9750 6300
-Wire Wire Line
-	9850 6000 9850 6300
-Wire Wire Line
-	9950 6000 9950 6300
 Text Label 8250 2350 0    50   ~ 0
 ~RST
@@
 	1    0    0    -1
 $EndComp
-Text Label 7050 4100 0    50   ~ 0
-CS_ICM
-Text Label 10650 5000 0    50   ~ 0
-DET_SD
 Wire Wire Line
 	2100 4300 3400 4300
