File: microbug/microbug.sch (KiCad schematic (older format))
At the start: 18 parts, among them J1 Conn_01x03, J2 Conn_01x03, M1 Motor_DC, M2 Motor_DC, U1 ATtiny1616-S, U2 QRE1113GR, U3 TC78H651AFNG, U4 QRE1113GR

Commit message: Added more LEDs, changed outline
Parts:
- added D2: LED, LED_THT:LED_D3.0mm, symbol Device:LED
- added D3: LED, LED_SMD:LED_0603_1608Metric_Pad1.05x0.95mm_HandSolder, symbol Device:LED
- added R6, R7: 220, Resistor_SMD:R_0603_1608Metric_Pad1.05x0.95mm_HandSolder, symbol Device:R
- added R8: 10k, Resistor_SMD:R_0603_1608Metric_Pad1.05x0.95mm_HandSolder, symbol Device:R
Connections:
- net +3V3: now also R8.1
- net GND: now also D2.1 (K), D3.1 (K)
- net UDPI: now also R8.2
- net LED3: now reaches U1.19 (PA3)
- net LED3: now also R7.1
- net LED2: now reaches U1.3 (PA5)
- net LED2: now also R6.1
- net LED renamed LED1
- new net: D2.2 (A), R6.2
- new net: D3.2 (A), R7.2
- no-connect marks 0 -> 6
Other:
- moved on the sheet: D1, J1, R1
Changed lines of the file:
@@
 L Connector_Generic:Conn_01x03 J1
 U 1 1 5E545F87
-P 2750 2950
-F 0 "J1" H 2668 2625 50  0000 C CNN
-F 1 "Conn_01x03" H 2668 2716 50  0000 C CNN
-F 2 "Connector_PinHeader_2.54mm:PinHeader_1x03_P2.54mm_Vertical" H 2750 2950 50  0001 C CNN
-F 3 "~" H 2750 2950 50  0001 C CNN
-	1    2750 2950
+P 2100 2950
+F 0 "J1" H 2018 2625 50  0000 C CNN
+F 1 "Conn_01x03" H 2018 2716 50  0000 C CNN
+F 2 "Connector_PinHeader_2.54mm:PinHeader_1x03_P2.54mm_Vertical" H 2100 2950 50  0001 C CNN
+F 3 "~" H 2100 2950 50  0001 C CNN
+	1    2100 2950
 	-1   0    0    1
 $EndComp
@@
 $EndComp
 Wire Wire Line
-	2950 3050 3100 3050
+	2300 3050 3100 3050
 Wire Wire Line
 	3100 3050 3100 3100
 Wire Wire Line
-	2950 2950 3150 2950
+	2300 2950 2550 2950
 $Comp
 L power:GND #PWR01
@@
 	3300 2500 3300 2850
 Wire Wire Line
-	2950 2850 3300 2850
+	2300 2850 3300 2850
 Wire Wire Line
 	3500 2500 3500 2700
-Text Notes 1800 3000 0    50   ~ 0
+Text Notes 1800 3250 0    50   ~ 0
 Programming Header
 Wire Notes Line
@@
 L Device:LED D1
 U 1 1 5E571E4A
-P 6750 5350
-F 0 "D1" V 6789 5233 50  0000 R CNN
-F 1 "LED" V 6698 5233 50  0000 R CNN
-F 2 "LED_SMD:LED_0603_1608Metric_Pad1.05x0.95mm_HandSolder" H 6750 5350 50  0001 C CNN
-F 3 "~" H 6750 5350 50  0001 C CNN
-	1    6750 5350
+P 4800 5450
+F 0 "D1" V 4839 5333 50  0000 R CNN
+F 1 "LED" V 4748 5333 50  0000 R CNN
+F 2 "LED_SMD:LED_0603_1608Metric_Pad1.05x0.95mm_HandSolder" H 4800 5450 50  0001 C CNN
+F 3 "~" H 4800 5450 50  0001 C CNN
+	1    4800 5450
 	0    -1   -1   0
 $EndComp
@@
 L power:GND #PWR07
 U 1 1 5E5747F3
-P 6750 5500
-F 0 "#PWR07" H 6750 5250 50  0001 C CNN
-F 1 "GND" H 6755 5327 50  0000 C CNN
-F 2 "" H 6750 5500 50  0001 C CNN
-F 3 "" H 6750 5500 50  0001 C CNN
-	1    6750 5500
+P 4800 5600
+F 0 "#PWR07" H 4800 5350 50  0001 C CNN
+F 1 "GND" H 4805 5427 50  0000 C CNN
+F 2 "" H 4800 5600 50  0001 C CNN
+F 3 "" H 4800 5600 50  0001 C CNN
+	1    4800 5600
 	1    0    0    -1
 $EndComp
@@
 L Device:R R1
 U 1 1 5E575B96
-P 6750 5050
-F 0 "R1" H 6820 5096 50  0000 L CNN
-F 1 "220" H 6820 5005 50  0000 L CNN
-F 2 "Resistor_SMD:R_0603_1608Metric_Pad1.05x0.95mm_HandSolder" V 6680 5050 50  0001 C CNN
-F 3 "~" H 6750 5050 50  0001 C CNN
-	1    6750 5050
+P 4800 5150
+F 0 "R1" H 4870 5196 50  0000 L CNN
+F 1 "220" H 4870 5105 50  0000 L CNN
+F 2 "Resistor_SMD:R_0603_1608Metric_Pad1.05x0.95mm_HandSolder" V 4730 5150 50  0001 C CNN
+F 3 "~" H 4800 5150 50  0001 C CNN
+	1    4800 5150
 	1    0    0    -1
 $EndComp
@@
 	6400 3950 6600 3950
 Wire Wire Line
-	6750 4900 6750 4800
+	4800 5000 4800 4900
 Text Label 6600 3150 0    50   ~ 0
-LED
-Text Label 6750 4800 0    50   ~ 0
-LED
+LED1
+Text Label 4800 4900 0    50   ~ 0
+LED1
 Text Label 6600 3850 0    50   ~ 0
 IR1
@@
 Wire Wire Line
 	3650 2500 3500 2500
+$Comp
+L Device:LED D2
+U 1 1 5E69F0F9
+P 5250 5450
+F 0 "D2" V 5289 5333 50  0000 R CNN
+F 1 "LED" V 5198 5333 50  0000 R CNN
+F 2 "LED_THT:LED_D3.0mm" H 5250 5450 50  0001 C CNN
+F 3 "~" H 5250 5450 50  0001 C CNN
+	1    5250 5450
+	0    -1   -1   0
+$EndComp
+$Comp
+L power:GND #PWR08
+U 1 1 5E69F0FF
+P 5250 5600
+F 0 "#PWR08" H 5250 5350 50  0001 C CNN
+F 1 "GND" H 5255 5427 50  0000 C CNN
+F 2 "" H 5250 5600 50  0001 C CNN
+F 3 "" H 5250 5600 50  0001 C CNN
+	1    5250 5600
+	1    0    0    -1
+$EndComp
+$Comp
+L Device:R R6
+U 1 1 5E69F105
+P 5250 5150
+F 0 "R6" H 5320 5196 50  0000 L CNN
+F 1 "220" H 5320 5105 50  0000 L CNN
+F 2 "Resistor_SMD:R_0603_1608Metric_Pad1.05x0.95mm_HandSolder" V 5180 5150 50  0001 C CNN
+F 3 "~" H 5250 5150 50  0001 C CNN
+	1    5250 5150
+	1    0    0    -1
+$EndComp
+Wire Wire Line
+	5250 5000 5250 4900
+Text Label 5250 4900 0    50   ~ 0
+LED2
+Text Label 6600 3250 0    50   ~ 0
+LED2
+Wire Wire Line
+	6400 3250 6600 3250
+Wire Wire Line
+	6400 3050 6600 3050
+Text Label 6600 3050 0    50   ~ 0
+LED3
+$Comp
+L Device:LED D3
+U 1 1 5E6CF7AC
+P 5700 5450
+F 0 "D3" V 5739 5333 50  0000 R CNN
+F 1 "LED" V 5648 5333 50  0000 R CNN
+F 2 "LED_SMD:LED_0603_1608Metric_Pad1.05x0.95mm_HandSolder" H 5700 5450 50  0001 C CNN
+F 3 "~" H 5700 5450 50  0001 C CNN
+	1    5700 5450
+	0    -1   -1   0
+$EndComp
+$Comp
+L power:GND #PWR0101
+U 1 1 5E6CF7B6
+P 5700 5600
+F 0 "#PWR0101" H 5700 5350 50  0001 C CNN
+F 1 "GND" H 5705 5427 50  0000 C CNN
+F 2 "" H 5700 5600 50  0001 C CNN
+F 3 "" H 5700 5600 50  0001 C CNN
+	1    5700 5600
+	1    0    0    -1
+$EndComp
+$Comp
+L Device:R R7
+U 1 1 5E6CF7C0
+P 5700 5150
+F 0 "R7" H 5770 5196 50  0000 L CNN
+F 1 "220" H 5770 5105 50  0000 L CNN
+F 2 "Resistor_SMD:R_0603_1608Metric_Pad1.05x0.95mm_HandSolder" V 5630 5150 50  0001 C CNN
+F 3 "~" H 5700 5150 50  0001 C CNN
+	1    5700 5150
+	1    0    0    -1
+$EndComp
+Wire Wire Line
+	5700 5000 5700 4900
+Text Label 5700 4900 0    50   ~ 0
+LED3
+NoConn ~ 6400 2850
+NoConn ~ 6400 2950
+NoConn ~ 6400 3350
+NoConn ~ 6400 3450
+NoConn ~ 6400 3650
+NoConn ~ 6400 3750
+$Comp
+L Device:R R8
+U 1 1 5E6EAF48
+P 2550 2550
+F 0 "R8" H 2620 2596 50  0000 L CNN
+F 1 "10k" H 2620 2505 50  0000 L CNN
+F 2 "Resistor_SMD:R_0603_1608Metric_Pad1.05x0.95mm_HandSolder" V 2480 2550 50  0001 C CNN
+F 3 "~" H 2550 2550 50  0001 C CNN
+	1    2550 2550
+	1    0    0    -1
+$EndComp
+Wire Wire Line
+	2550 2700 2550 2950
+Connection ~ 2550 2950
+Wire Wire Line
+	2550 2950 3150 2950
+$Comp
+L power:+3.3V #PWR0102
+U 1 1 5E6ED31E
+P 2550 2400
+F 0 "#PWR0102" H 2550 2250 50  0001 C CNN
+F 1 "+3.3V" H 2565 2573 50  0000 C CNN
+F 2 "" H 2550 2400 50  0001 C CNN
+F 3 "" H 2550 2400 50  0001 C CNN
+	1    2550 2400
+	1    0    0    -1
+$EndComp
 $EndSCHEMATC

Commit message: microbug bugging
Parts:
- added J3: Conn_01x02, Connector_PinHeader_2.54mm:PinHeader_1x02_P2.54mm_Vertical, symbol Connector_Generic:Conn_01x02
- M1, M2: footprint Connector_PinHeader_2.54mm:PinHeader_1x02_P2.54mm_Vertical -> microbug-fplib:micro_motor_5mm
- U1: symbol MCU_Microchip_ATtiny:ATtiny1616-S -> microbug-rescue:ATtiny1616-S-MCU_Microchip_ATtiny
Connections:
- net GND: now also J3.1 (Pin_1)
- net LED1: now also U1.10 (PB1); no longer U1.2 (PA4)
- net LED3: now also U1.11 (PB0); no longer U1.19 (PA3)
- net UDPI: now also J1.3 (Pin_3); no longer J1.2 (Pin_2)
- net SDA: now reaches U1.17 (PA1)
- net SCL: now reaches U1.18 (PA2)
- net DAC: now reaches U1.4 (PA6)
- net DAC: now also J3.2 (Pin_2)
- net at M1.1 (+): now also U3.11 (OUT2); no longer U3.12 (OUT1)
- net at M1.2 (-): now also U3.12 (OUT1); no longer U3.11 (OUT2)
- net at M2.1 (+): now also U3.15 (OUT4); no longer U3.14 (OUT3)
- net at M2.2 (-): now also U3.14 (OUT3); no longer U3.15 (OUT4)
- net at J2.3 (Pin_3): now also J1.2 (Pin_2); no longer J1.3 (Pin_3)
- no-connect marks 6 -> 3
Other:
- note added: "Extra Pinout"
- note added: "LEDs"
- moved on the sheet: D1, D2, D3, R1, R6, R7, R8
