File: microbug/microbug.kicad_sch (KiCad schematic)
At the start: 26 parts, among them J1 Conn_01x04, J2 Conn_01x03, J3 Conn_01x02, M1 Motor_DC, M2 Motor_DC, U1 ATtiny1616-S, U2 QRE1113GR, U3 QRE1113GR, U5 TC78H660FNG

Commit message: new layout edits, still missing logo
Parts:
- D1, D3: footprint LED_SMD:LED_0603_1608Metric_Pad1.05x0.95mm_HandSolder -> LED_THT:LED_D3.0mm
Connections:
- net at M2.1 (+): now also U5.9 (OUTB-); no longer U5.10 (OUTB+)
- net at M2.2 (-): now also U5.10 (OUTB+); no longer U5.9 (OUTB-)
Other:
- moved on the sheet: M2
Changed lines of the file:
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@@
       (effects (font (size 1.27 1.27)) (justify right))
     )
-    (property "Footprint" "LED_SMD:LED_0603_1608Metric_Pad1.05x0.95mm_HandSolder" (id 2) (at 135.89 142.24 0)
+    (property "Footprint" "LED_THT:LED_D3.0mm" (id 2) (at 135.89 142.24 0)
       (effects (font (size 1.27 1.27)) hide)
     )
@@
       (effects (font (size 1.27 1.27)) (justify right))
     )
-    (property "Footprint" "LED_SMD:LED_0603_1608Metric_Pad1.05x0.95mm_HandSolder" (id 2) (at 158.75 142.24 0)
+    (property "Footprint" "LED_THT:LED_D3.0mm" (id 2) (at 158.75 142.24 0)
       (effects (font (size 1.27 1.27)) hide)
     )
@@
     (pin "4")
   )
-  (symbol (lib_id "Motor:Motor_DC") (at 240.03 87.63 0) (mirror y) (unit 1)
-    (in_bom yes) (on_board yes)
-    (property "Reference" "M2" (id 0) (at 246.5578 89.7636 0)
-      (effects (font (size 1.27 1.27)) (justify left))
-    )
-    (property "Value" "Motor_DC" (id 1) (at 252.3998 87.63 0)
-      (effects (font (size 1.27 1.27)) (justify left))
-    )
-    (property "Footprint" "microbug-fplib:micro_motor_5mm" (id 2) (at 240.03 89.916 0)
-      (effects (font (size 1.27 1.27)) hide)
-    )
-    (property "Datasheet" "~" (id 3) (at 240.03 89.916 0)
+  (symbol (lib_id "Motor:Motor_DC") (at 240.03 90.17 180) (unit 1)
+    (in_bom yes) (on_board yes)
+    (property "Reference" "M2" (id 0) (at 246.5578 88.0364 0)
+      (effects (font (size 1.27 1.27)) (justify left))
+    )
+    (property "Value" "Motor_DC" (id 1) (at 252.3998 90.17 0)
+      (effects (font (size 1.27 1.27)) (justify left))
+    )
+    (property "Footprint" "microbug-fplib:micro_motor_5mm" (id 2) (at 240.03 87.884 0)
+      (effects (font (size 1.27 1.27)) hide)
+    )
+    (property "Datasheet" "~" (id 3) (at 240.03 87.884 0)
       (effects (font (size 1.27 1.27)) hide)
     )
@@
     )
     (path "/00000000-0000-0000-0000-00005e571e4a"
-      (reference "D1") (unit 1) (value "LED") (footprint "LED_SMD:LED_0603_1608Metric_Pad1.05x0.95mm_HandSolder")
+      (reference "D1") (unit 1) (value "LED") (footprint "LED_THT:LED_D3.0mm")
     )
     (path "/00000000-0000-0000-0000-00005e69f0f9"
@@
     )
     (path "/00000000-0000-0000-0000-00005e6cf7ac"
-      (reference "D3") (unit 1) (value "LED") (footprint "LED_SMD:LED_0603_1608Metric_Pad1.05x0.95mm_HandSolder")
+      (reference "D3") (unit 1) (value "LED") (footprint "LED_THT:LED_D3.0mm")
     )
     (path "/8951631c-7a8e-4f41-b6ed-40b357def0bf"

Commit message: bug gets new connector, logo silk, small changes
Parts:
- added J4: Conn_01x02, Connector_PinHeader_2.54mm:PinHeader_1x02_P2.54mm_Vertical, symbol Connector_Generic:Conn_01x02
Connections:
- net +3V3: now also U5.14 (STBY); no longer U5.15 (MODE/ERR)
- net GND: now also J4.1 (Pin_1)
- net V_bat: now reaches BT1.1 (+), J2.1 (Pin_1)
- net V_bat: now also J4.2 (Pin_2)
- net at R10.2: now also U5.15 (MODE/ERR); no longer U5.14 (STBY)
Other:
- moved on the sheet: C2, C3, M1, M2, R10, R9, U5
